File: KiCADProjects/WaterChangeCircuits/WaterChangeCircuits.kicad_pcb (KiCad board)
At the start: 2 copper layers, 122 parts, among them J1 Conn_01x25, J10 Conn_01x02, J11 Conn_01x02, J12 Conn_01x02, J13 Conn_01x02, J14 Conn_01x02, J15 Conn_01x02, J16 Conn_01x02, J17 Conn_01x02, J18 Conn_01x02, J19 Conn_01x02, J2 Conn_01x27, J20 Conn_01x02, J21 Conn_01x02, J22 Conn_01x02, J23 Conn_01x02, J24 Conn_01x02, J25 Conn_01x02, J26 Conn_01x02, J27 Conn_01x02, J28 Conn_01x02, J29 Conn_01x02, J3 Conn_01x02, J30 Conn_01x02, J31 Conn_01x02, J32 Conn_01x02, J33 Conn_01x02, J34 Conn_01x02, J35 Conn_01x02, J36 Conn_01x02, J37 Conn_01x02, J38 Conn_01x02, J39 Conn_01x02, J4 Conn_01x02, J40 Conn_01x02, J41 Conn_01x02, J42 Conn_01x02, J43 Conn_01x02, J44 Conn_01x02, J45 Conn_01x02, J46 Conn_01x02, J47 Conn_01x02, J48 Conn_01x02, J49 Conn_01x02, J5 Conn_01x02, J50 Conn_01x02, J51 Conn_01x02, J52 Conn_01x02, J53 Conn_01x02, J54 Barrel_Jack, J55 Conn_02x02_Odd_Even, J56 Conn_01x02, J57 Conn_01x16, J58 Conn_01x03, J59 Conn_01x03, J6 Conn_01x02, J60 Conn_01x03, J61 Conn_01x03, J62 Conn_01x03, J63 Conn_01x03, J64 Conn_01x03, J65 Conn_01x03, J66 Conn_01x03, J67 Conn_01x03, J68 Conn_01x03, J69 Conn_01x03, J7 Conn_01x02, J70 Conn_01x03, J71 Conn_01x03, J72 Conn_01x03, J73 Conn_01x03, J8 Conn_01x02, J9 Conn_01x02, U1 TLP3542, U10 TLP3542, U11 TLP3542, U12 TLP3542, U13 TLP3542, U14 TLP3542, U15 TLP3542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

Commit message: Completed PCB design and schematics.
Parts:
- removed U10, U11, U12, U13, U6, U7, U8, U9: TLP3542, Package_DIP:DIP-5-6_W7.62mm
- added H1: MountingHole, MountingHole:MountingHole_3.2mm_M3, F.Cu at (-26.7, 84.6)
- added H2: MountingHole, MountingHole:MountingHole_3.2mm_M3, F.Cu at (-26.5, 124.2)
- added H3: MountingHole, MountingHole:MountingHole_3.2mm_M3, F.Cu at (339.6, 84.6)
- added H4: MountingHole, MountingHole:MountingHole_3.2mm_M3, F.Cu at (341.4, 125.9)
- added J74: Conn_01x03, Connector_PinSocket_2.54mm:PinSocket_1x03_P2.54mm_Vertical, F.Cu at (266.2, 84.1)
- added J75: Conn_01x03, Connector_PinSocket_2.54mm:PinSocket_1x03_P2.54mm_Vertical, F.Cu at (257.3, 84.1)
- J10, J11, J13, J14, J15, J16, J17: value Conn_01x02 -> Conn_01x03; footprint Connector_JST:JST_PH_S2B-PH-K_1x02_P2.00mm_Horizontal -> Connector_PinSocket_2.54mm:PinSocket_1x03_P2.54mm_Vertical
- J12: value Conn_01x02 -> Conn_01x12; footprint Connector_JST:JST_PH_S2B-PH-K_1x02_P2.00mm_Horizontal -> Connector_PinSocket_2.54mm:PinSocket_1x12_P2.54mm_Vertical
- J2: value Conn_01x27 -> Conn_01x15; footprint Connector_PinSocket_2.54mm:PinSocket_1x27_P2.54mm_Vertical -> Connector_PinSocket_2.54mm:PinSocket_1x15_P2.54mm_Vertical
- J54: value Barrel_Jack -> Barrel_Jack_Switch
- moved J53 302.1 mm to (-32.9, 153.3)
- moved J51 255.8 mm to (-14.4, 153.3)
- moved J1 248.4 mm to (272.0, 114.7), turned to 90 degrees
- moved J46 218.5 mm to (32.0, 153.3)
- moved J52 213.6 mm to (-23.6, 153.3)
- moved J44 208.4 mm to (50.5, 153.3)
- moved J43 205.2 mm to (59.8, 153.3)
- moved J47 202.1 mm to (22.7, 153.3)
- moved J48 201.8 mm to (13.5, 153.3)
- moved J49 199.0 mm to (4.19, 153.3)
- moved U38 197.8 mm to (74.2, 139.7), turned to 270 degrees
- moved J50 196.7 mm to (-5.08, 153.3)
- moved J45 196.6 mm to (41.3, 153.3)
- moved J12 195.7 mm to (17.3, 114.4), turned to 90 degrees
- moved U44 182.7 mm to (18.5, 139.8), turned to 270 degrees
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Connections:
- J10 pad 1: T1 -> +5V
- J10 pad 2: GND1 -> D13
- J11 pad 1: T2 -> +5V
- J11 pad 2: GND1 -> D12
- J12 pad 1: T3 -> D53
- J12 pad 2: GND1 -> D52
- J13 pad 1: T4 -> +5V
- J13 pad 2: GND1 -> D11
- J14 pad 1: T5 -> +5V
- J14 pad 2: GND1 -> D10
- J15 pad 1: T6 -> +5V
- J15 pad 2: GND1 -> D09
- J16 pad 1: T7 -> +5V
- J16 pad 2: GND1 -> D14
- J17 pad 1: T8 -> +5V
- J17 pad 2: GND1 -> D15
- J2 pad 1: D53 -> D41
- J2 pad 10: D44 -> D32
- J2 pad 11: D43 -> D31
- J2 pad 12: D42 -> D30
- J2 pad 13: D41 -> D29
- J2 pad 14: D40 -> D28
- J2 pad 15: D39 -> D27
- J2 pad 2: D52 -> D40
- J2 pad 3: D51 -> D39
- J2 pad 4: D50 -> D38
- J2 pad 5: D49 -> D37
- J2 pad 6: D48 -> D36
- J2 pad 7: D47 -> D35
- J2 pad 8: D46 -> D34
- J2 pad 9: D45 -> D33
- J54 pad 3: (no net) -> GND1
Routing:
- net GND2: track 200.3 -> 1103.7 mm
- net GND1: track 18.2 -> 573.0 mm
- net +12V: track 18.8 -> 529.6 mm
- net +5V: track 2.54 -> 463.8 mm
- net A15: track 0.00 -> 130.4 mm
- net A14: track 0.00 -> 125.5 mm
- net A13: track 0.00 -> 118.2 mm
- net A12: track 0.00 -> 110.2 mm
- net A11: track 0.00 -> 102.7 mm
- net A10: track 0.00 -> 95.7 mm
- net D41: track 0.00 -> 90.3 mm
- net A9: track 0.00 -> 88.8 mm
- net D40: track 0.00 -> 83.5 mm
- net A8: track 0.00 -> 82.0 mm
- net D39: track 0.00 -> 76.8 mm
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Other:
- board outline added: 380.7 x 79.6 mm
- rule pad_to_mask_clearance: 0 -> 0.0508
- board text added: "Analog Pins"
- board text added: "D02"
- board text added: "D26"
- board text added: "D27"
- board text added: "D41"
- board text added: "D42"
- board text added: "D53"
- board text added: "Digital Pins 26-02"
- board text added: "Digital Pins 41-27"
- board text added: "Digital Pins 53-42"
- board text added: "Float Switches"
- board text added: "Flow Meters"
- board text added: "To Pi +5V"
- board text added: "To Pi GND"

Commit message: Added PDF of the schematic
Other:
- rule trace_min: 0.2 -> 0.1524
- rule via_min_drill: 0.3 -> 0.254
- rule via_min_size: 0.4 -> 0.508

Commit message: Updated some design files and added parts of the web app
Parts:
- moved J54 9.00 mm to (-25.1, 99.9), turned to 270 degrees
- moved J56 7.31 mm to (-25.7, 109.6), turned to 270 degrees
- moved H1 3.51 mm to (-29.0, 87.2)
- moved H2 2.50 mm to (-29.0, 124.8)
Routing:
- net GND1: track 573.0 -> 571.6 mm
- net +12V: track 529.6 -> 530.7 mm
Other:
- board text added: "+12v"
- board text added: "+5v"
- board text added: "12v GND"
- board text added: "5v GND"
